File: PhysicsClubDemo/PhysicsClubDemo.kicad_sch (KiCad schematic)
At the start: 11 parts, among them U1 OFF, U2 Analog_1, U3 Analog_2, U4 ESP32-S3, U5 ICSP, U6 Digital_1, U7 Digital_2

Commit message: First commit !
Other:
- note added: "Schematic - Component Placement"
- note removed: "Arduino UNO R4 Shield"
- company: MStackoverflow -> Victor Rosales
- title: Arduino UNO R4 Shield Template SCH -> Electric Components Demo
- moved on the sheet: H1, H2, H3, H4, U1, U2, U3, U4, U5, U6, U7
